File: zero-cam.kicad_pcb (KiCad board)
At the start: 2 copper layers, 140 x 45 mm, 87 parts, among them J1 DC 12-24V, J2 Conn_01x04, J3 Front_Plate, J4 Edge_Connector, Q1 tbd, Q2 tbd, U1 LMR36510, U2 Raspberry_Pi_ZeroW, U3 LP2985-3.3, U4 M24C02-FDW, U5 BME280, U6 ARJM11D7-114, U7 ENC424J600-PT, Y1 25MHz 50ppm

Commit message: Layout almost done
Parts:
- added C28: 2.2uF, Capacitor_SMD:C_1210_3225Metric_Pad1.33x2.70mm_HandSolder, F.Cu at (110.2, 73.0)
- added D12: IR, LED_SMD:LED_0805_2012Metric_Pad1.15x1.40mm_HandSolder, F.Cu at (185.2, 83.8)
- added D13: IR, LED_SMD:LED_0805_2012Metric_Pad1.15x1.40mm_HandSolder, F.Cu at (188.7, 77.2)
- added D14: IR, LED_SMD:LED_0805_2012Metric_Pad1.15x1.40mm_HandSolder, F.Cu at (185.2, 91.0)
- added D15: IR, LED_SMD:LED_0805_2012Metric_Pad1.15x1.40mm_HandSolder, F.Cu at (188.7, 97.8)
- added R22: 100R, Resistor_SMD:R_0805_2012Metric_Pad1.20x1.40mm_HandSolder, F.Cu at (191.5, 72.8)
- added R23: 100R, Resistor_SMD:R_0805_2012Metric_Pad1.20x1.40mm_HandSolder, F.Cu at (191.5, 102.2)
- J3: value Front_Plate -> Edge_Connector; footprint Connector_PinSocket_2.54mm:PinSocket_2x05_P2.54mm_Vertical -> zero-cam:Edge_PinHeader_2x05_P2; moved to F.Cu
- J4: value Edge_Connector -> Front_Plate; footprint zero-cam:Edge_PinHeader_2x05_P2 -> Connector_PinSocket_2.54mm:PinSocket_2x05_P2.54mm_Vertical; moved to B.Cu
- moved J3 18.3 mm to (166.5, 87.5)
- moved R5 16.3 mm to (210.0, 104.5)
- moved J4 16.0 mm to (181.8, 92.5)
- moved R4 12.0 mm to (208.0, 70.5)
- moved D8 9.33 mm to (203.8, 102.2), turned to 90 degrees
- moved D2 8.78 mm to (203.8, 72.8), turned to 270 degrees
- moved Q2 7.81 mm to (182.5, 99.0), turned to 180 degrees
- moved R1 7.10 mm to (183.0, 79.5)
- moved FID3 6.04 mm to (215.0, 76.0)
- moved D3 5.47 mm to (197.2, 72.5), turned to 270 degrees
- moved Q1 5.03 mm to (182.8, 76.0), turned to 180 degrees
- moved FID4 4.92 mm to (187.0, 102.0)
- moved D9 4.70 mm to (197.2, 102.5), turned to 90 degrees
- moved D7 4.61 mm to (210.0, 99.0)
- moved D4 4.42 mm to (213.2, 80.0)
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Connections:
- J3 pad 2: L_SENSE -> +5V
- J3 pad 3: PWM_1 -> L_SENSE
- J3 pad 4: PWM_0 -> Net-(J3-Pad4)
- J3 pad 5: GND -> PWM_1
- J3 pad 6: +5V -> Net-(J3-Pad6)
- J3 pad 7: (no net) -> PWM_0
- J3 pad 8: (no net) -> Net-(J3-Pad8)
- J3 pad 9: (no net) -> GND
- J4 pad 2: L_SENSE -> +5V
- J4 pad 3: PWM_1 -> L_SENSE
- J4 pad 4: PWM_0 -> Net-(J4-Pad4)
- J4 pad 5: GND -> PWM_1
- J4 pad 6: +5V -> Net-(J4-Pad6)
- J4 pad 7: (no net) -> PWM_0
- J4 pad 8: (no net) -> Net-(J4-Pad8)
- J4 pad 9: (no net) -> GND
- U2 pad 12: (no net) -> Net-(U2-Pad12)
- U2 pad 13: (no net) -> Net-(U2-Pad13)
- U2 pad 16: (no net) -> PWM_0
- U2 pad 18: (no net) -> PWM_1
- U2 pad 22: (no net) -> L_SENSE
- U2 pad 26: (no net) -> Net-(U2-Pad26)
- U2 pad 29: (no net) -> Net-(U2-Pad29)
- U2 pad 31: (no net) -> Net-(U2-Pad31)
- U2 pad 32: PWM_0 -> Net-(U2-Pad32)
- U2 pad 33: PWM_1 -> Net-(U2-Pad33)
- U2 pad 35: (no net) -> Net-(U2-Pad35)
- U2 pad 36: (no net) -> Net-(U2-Pad36)
- U2 pad 37: L_SENSE -> Net-(U2-Pad37)
- U2 pad 38: (no net) -> Net-(U2-Pad38)
- U2 pad 40: (no net) -> Net-(U2-Pad40)
- U7 pad 23: (no net) -> E_CLK_OUT
- U7 pad 25: (no net) -> Net-(U7-Pad25)
- U7 pad 26: (no net) -> Net-(U7-Pad26)
- U7 pad 27: (no net) -> Net-(U7-Pad27)
- U7 pad 28: (no net) -> Net-(U7-Pad28)
- U7 pad 29: (no net) -> Net-(U7-Pad29)
- U7 pad 30: (no net) -> Net-(U7-Pad30)
- U7 pad 31: (no net) -> Net-(U7-Pad31)
- U7 pad 32: (no net) -> Net-(U7-Pad32)
- U7 pad 38: (no net) -> Net-(U7-Pad38)
- U7 pad 39: (no net) -> Net-(U7-Pad39)
- U7 pad 40: (no net) -> Net-(U7-Pad40)
- U7 pad 41: (no net) -> Net-(U7-Pad41)
- U7 pad 5: (no net) -> Net-(U7-Pad5)
- U7 pad 6: (no net) -> Net-(U7-Pad6)
- U7 pad 7: (no net) -> Net-(U7-Pad7)
- U7 pad 8: (no net) -> Net-(U7-Pad8)
Routing:
- net +5V: track 29.5 -> 157.6 mm, vias 4 -> 10
- net L_SENSE: track 0.00 -> 98.2 mm
- net PWM_1: track 0.00 -> 61.8 mm
- net PWM_0: track 0.00 -> 58.2 mm
- net POE-: track 0.00 -> 51.4 mm
- net /ethernet_if/led_a: track 0.00 -> 49.0 mm, vias 0 -> 2
- net /ethernet_if/led_b: track 1.50 -> 33.3 mm, vias 0 -> 2
- net Net-(Q2-Pad1): track 0.00 -> 31.1 mm
- net Net-(Q1-Pad1): track 0.00 -> 28.3 mm
- net Net-(D11-Pad2): track 0.00 -> 25.7 mm
- net Net-(D10-Pad2): track 0.00 -> 16.5 mm
- net Net-(C19-Pad1): track 3.94 -> 19.7 mm
- net /pg: track 0.00 -> 12.3 mm
- net Net-(D12-Pad1): track 0.00 -> 9.81 mm
- net Net-(D14-Pad1): track 0.00 -> 9.76 mm
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Other:
- outline, holes or cut-outs redrawn

Commit message: Release v0.2.0
Parts:
- J2: value Conn_01x04 -> Conn_01x03; footprint Connector_PinHeader_2.00mm:PinHeader_1x04_P2.00mm_Vertical -> Connector_PinHeader_2.54mm:PinHeader_1x03_P2.54mm_Vertical
- moved C17 17.4 mm to (168.0, 75.0), turned to 270 degrees
- moved U5 15.3 mm to (165.0, 75.0), turned to 90 degrees
- moved C27 3.51 mm to (110.0, 86.2)
- moved C18 2.00 mm to (143.8, 88.0), turned to 90 degrees
- moved J2 1.82 mm to (118.2, 104.8)
Connections:
- J2 pad 1: +3.3VA -> Net-(J2-Pad1)
- J2 pad 3: Net-(J2-Pad3) -> GND
- U2 pad 10: Net-(J2-Pad2) -> Net-(J2-Pad1)
- U2 pad 8: Net-(J2-Pad3) -> Net-(J2-Pad2)
Routing:
- net SDA_1: track 0.00 -> 71.6 mm, vias 0 -> 1
- net SCL_1: track 0.00 -> 69.2 mm, vias 0 -> 1
- net +3.3VA: track 2.98 -> 69.4 mm, vias 0 -> 3
- net GND: track 34.7 -> 91.1 mm, vias 19 -> 115
- net +3V3: track 33.4 -> 76.6 mm, vias 0 -> 4
- net +5V: track 157.6 -> 199.5 mm, vias 10 -> 15
- net PWR_GOOD: track 0.00 -> 37.5 mm, vias 0 -> 1
- net E_OFF: track 2.17 -> 23.0 mm, vias 0 -> 1
- net HAT_SDA: track 0.00 -> 11.6 mm
- net HAT_SCL: track 4.64 -> 14.0 mm
- net /WC: track 0.00 -> 6.10 mm
- net Net-(J2-Pad2): track 0.00 -> 4.65 mm
- net Net-(J2-Pad1): track 0.00 -> 4.65 mm
- net /ethernet_if/led_a: track 49.0 -> 49.8 mm
- net /ethernet_if/TP_OUT+: track 25.1 -> 24.5 mm
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Other:
- board text added: "Zero-Cam, v0.2.0 May 2021"
- board text added: "github.com/juraj8/zero-cam"
