File: zero-cam.sch (KiCad schematic (older format))
At the start: 48 parts, among them J2 DC 12-24V, J4 Conn_01x04, Q1 tbd, Q2 tbd, U1 LMR36510, U2 Raspberry_Pi_ZeroW, U3 LP2985-3.3, U4 M24C02-FDW, U5 BME280

Commit message: Change for actual footprints, raff  board done.
Parts:
- added C13: 0.1uF, Capacitor_SMD:C_0603_1608Metric_Pad1.08x0.95mm_HandSolder, symbol Device:C_Small
- added R7: 10k, Resistor_SMD:R_0805_2012Metric_Pad1.20x1.40mm_HandSolder, symbol Device:R_Small
- C1: footprint Capacitor_SMD:C_0805_2012Metric_Pad1.18x1.45mm_HandSolder -> Capacitor_SMD:C_1210_3225Metric_Pad1.33x2.70mm_HandSolder
- C11: renamed from C10; footprint Capacitor_SMD:C_0805_2012Metric_Pad1.18x1.45mm_HandSolder -> Capacitor_SMD:C_1206_3216Metric_Pad1.33x1.80mm_HandSolder
- C8: renamed from C7; footprint Capacitor_SMD:C_0805_2012Metric_Pad1.18x1.45mm_HandSolder -> Capacitor_SMD:C_1206_3216Metric_Pad1.33x1.80mm_HandSolder
- C9: renamed from C8; footprint Capacitor_SMD:C_0805_2012Metric_Pad1.18x1.45mm_HandSolder -> Capacitor_SMD:C_1206_3216Metric_Pad1.33x1.80mm_HandSolder
- D1: value tbd -> B160-13-F; footprint LED_SMD:LED_0805_2012Metric_Pad1.15x1.40mm_HandSolder -> Diode_SMD:D_SMA_Handsoldering
- J1: renamed from J2; footprint Connector_BarrelJack:BarrelJack_Wuerth_6941xx301002 -> Connector_BarrelJack:BarrelJack_Horizontal
- L1: footprint Inductor_SMD:L_Wuerth_HCM-1350 -> Inductor_SMD:L_10.4x10.4_H4.8
- renumbered C9 to C10, C13 to C14, C14 to C15, C15 to C16, C16 to C17, C17 to C18, C11 to C5, C5 to C6, C6 to C7, J4 to J2, R4 to R10, R5 to R11, R11 to R12, R6 to R4, R7 to R5, R8 to R6, R9 to R8, R10 to R9
Connections:
- wire segments 202 -> 203

Commit message: Connector placment done, dimentions decided ...
Parts:
- added FID1, FID2, FID3, FID4: Fiducial, Fiducial:Fiducial_0.5mm_Mask1mm, symbol Mechanical:Fiducial
- added H1, H2, H3, H4, H5, H6, H7, H8: MountingHole, MountingHole:MountingHole_3.2mm_M3_DIN965, symbol Mechanical:MountingHole
- added J3: Conn_02x05_Top_Bottom, Connector_PinSocket_2.54mm:PinSocket_2x05_P2.54mm_Vertical, symbol Connector_Generic:Conn_02x05_Top_Bottom
- added J4: Conn_02x05_Top_Bottom, zero-cam:Edge_PinHeader_2x05_P2, symbol Connector_Generic:Conn_02x05_Top_Bottom
Connections:
- net labels added: WC, boot, fb, pg, sw
- wire segments 203 -> 209
Other:
- moved on the sheet: C15, C17, C5, D2, D3, D4, D5, D6, D7, D8, D9, JP1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

Commit message: start layout
Parts:
- J3: value Conn_02x05_Top_Bottom -> Front_Plate
- J4: value Conn_02x05_Top_Bottom -> Edge_Connector
Connections:
- wire segments 209 -> 225
- no-connect marks 13 -> 19
Changed lines of the file:
@@
 P 3050 7000
 F 0 "J3" H 3100 7417 50  0000 C CNN
-F 1 "Conn_02x05_Top_Bottom" H 3100 7326 50  0000 C CNN
+F 1 "Front_Plate" H 3100 7326 50  0000 C CNN
 F 2 "Connector_PinSocket_2.54mm:PinSocket_2x05_P2.54mm_Vertical" H 3050 7000 50  0001 C CNN
 F 3 "~" H 3050 7000 50  0001 C CNN
@@
 P 1400 7000
 F 0 "J4" H 1450 7417 50  0000 C CNN
-F 1 "Conn_02x05_Top_Bottom" H 1450 7326 50  0000 C CNN
+F 1 "Edge_Connector" H 1450 7326 50  0000 C CNN
 F 2 "zero-cam:Edge_PinHeader_2x05_P2" H 1400 7000 50  0001 C CNN
 F 3 "~" H 1400 7000 50  0001 C CNN
@@
 Text Label 8150 3050 0    11   ~ 0
 WC
+$Comp
+L power:GND #PWR0101
+U 1 1 608CEF28
+P 1100 7300
+F 0 "#PWR0101" H 1100 7050 50  0001 C CNN
+F 1 "GND" V 1105 7172 50  0000 R CNN
+F 2 "" H 1100 7300 50  0001 C CNN
+F 3 "" H 1100 7300 50  0001 C CNN
+	1    1100 7300
+	-1   0    0    -1
+$EndComp
+Wire Wire Line
+	1200 7200 1100 7200
+Wire Wire Line
+	1100 7200 1100 7300
+$Comp
+L power:GND #PWR0102
+U 1 1 608DAC30
+P 2750 7300
+F 0 "#PWR0102" H 2750 7050 50  0001 C CNN
+F 1 "GND" V 2755 7172 50  0000 R CNN
+F 2 "" H 2750 7300 50  0001 C CNN
+F 3 "" H 2750 7300 50  0001 C CNN
+	1    2750 7300
+	-1   0    0    -1
+$EndComp
+Wire Wire Line
+	2850 7200 2750 7200
+Wire Wire Line
+	2750 7200 2750 7300
+Text GLabel 1200 7100 0    50   Input ~ 0
+PWM_0
+Text GLabel 1200 7000 0    50   Input ~ 0
+PWM_1
+Text GLabel 2850 7000 0    50   Input ~ 0
+PWM_1
+Text GLabel 2850 7100 0    50   Input ~ 0
+PWM_0
+Text GLabel 1200 6900 0    50   Output ~ 0
+L_SENSE
+Text GLabel 2850 6900 0    50   Output ~ 0
+L_SENSE
+$Comp
+L power:+5V #PWR0103
+U 1 1 608E6D85
+P 1100 6700
+F 0 "#PWR0103" H 1100 6550 50  0001 C CNN
+F 1 "+5V" H 1115 6873 50  0000 C CNN
+F 2 "" H 1100 6700 50  0001 C CNN
+F 3 "" H 1100 6700 50  0001 C CNN
+	1    1100 6700
+	-1   0    0    -1
+$EndComp
+Wire Wire Line
+	1100 6700 1100 6800
+Wire Wire Line
+	1100 6800 1200 6800
+$Comp
+L power:+5V #PWR0104
+U 1 1 608F34F1
+P 2750 6700
+F 0 "#PWR0104" H 2750 6550 50  0001 C CNN
+F 1 "+5V" H 2765 6873 50  0000 C CNN
+F 2 "" H 2750 6700 50  0001 C CNN
+F 3 "" H 2750 6700 50  0001 C CNN
+	1    2750 6700
+	-1   0    0    -1
+$EndComp
+Wire Wire Line
+	2750 6700 2750 6800
+Wire Wire Line
+	2750 6800 2850 6800
+$Comp
+L power:+5V #PWR?
+U 1 1 6090443A
+P 3500 6700
+F 0 "#PWR?" H 3500 6550 50  0001 C CNN
+F 1 "+5V" H 3515 6873 50  0000 C CNN
+F 2 "" H 3500 6700 50  0001 C CNN
+F 3 "" H 3500 6700 50  0001 C CNN
+	1    3500 6700
+	-1   0    0    -1
+$EndComp
+Wire Wire Line
+	3350 6800 3500 6800
+Wire Wire Line
+	3500 6800 3500 6700
+$Comp
+L power:GND #PWR?
+U 1 1 60910A1B
+P 3500 7300
+F 0 "#PWR?" H 3500 7050 50  0001 C CNN
+F 1 "GND" V 3505 7172 50  0000 R CNN
+F 2 "" H 3500 7300 50  0001 C CNN
+F 3 "" H 3500 7300 50  0001 C CNN
+	1    3500 7300
+	-1   0    0    -1
+$EndComp
+Wire Wire Line
+	3350 7200 3500 7200
+Wire Wire Line
+	3500 7200 3500 7300
+$Comp
+L power:+5V #PWR?
+U 1 1 6091E285
+P 1800 6700
+F 0 "#PWR?" H 1800 6550 50  0001 C CNN
+F 1 "+5V" H 1815 6873 50  0000 C CNN
+F 2 "" H 1800 6700 50  0001 C CNN
+F 3 "" H 1800 6700 50  0001 C CNN
+	1    1800 6700
+	-1   0    0    -1
+$EndComp
+Wire Wire Line
+	1800 6700 1800 6800
+Wire Wire Line
+	1800 6800 1700 6800
+$Comp
+L power:GND #PWR?
+U 1 1 6092BCCF
+P 1800 7300
+F 0 "#PWR?" H 1800 7050 50  0001 C CNN
+F 1 "GND" V 1805 7172 50  0000 R CNN
+F 2 "" H 1800 7300 50  0001 C CNN
+F 3 "" H 1800 7300 50  0001 C CNN
+	1    1800 7300
+	-1   0    0    -1
+$EndComp
+Wire Wire Line
+	1700 7200 1800 7200
+Wire Wire Line
+	1800 7200 1800 7300
+NoConn ~ 1700 6900
+NoConn ~ 1700 7000
+NoConn ~ 1700 7100
+NoConn ~ 3350 6900
+NoConn ~ 3350 7000
+NoConn ~ 3350 7100
 $EndSCHEMATC

Commit message: Layout almost done
Parts:
- removed J3: Front_Plate, Connector_PinSocket_2.54mm:PinSocket_2x05_P2.54mm_Vertical, symbol Connector_Generic:Conn_02x05_Top_Bottom
- removed J4: Edge_Connector, zero-cam:Edge_PinHeader_2x05_P2, symbol Connector_Generic:Conn_02x05_Top_Bottom
- added C28: 2.2uF, Capacitor_SMD:C_1210_3225Metric_Pad1.33x2.70mm_HandSolder, symbol Device:C_Small
- added D12, D13, D14, D15: IR, LED_SMD:LED_0805_2012Metric_Pad1.15x1.40mm_HandSolder, symbol Device:LED_Small
- added J3: Edge_Connector, zero-cam:Edge_PinHeader_2x05_P2, symbol Connector_Generic:Conn_02x05_Odd_Even
- added J4: Front_Plate, Connector_PinSocket_2.54mm:PinSocket_2x05_P2.54mm_Vertical, symbol Connector_Generic:Conn_02x05_Odd_Even
- added R22, R23: 100R, Resistor_SMD:R_0805_2012Metric_Pad1.20x1.40mm_HandSolder, symbol Device:R_Small
Connections:
- wire segments 225 -> 235
Other:
- moved on the sheet: C1, C2, D1, D2, D3, D4, D5, Q1, Q2, R1, R2, R3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

Commit message: Release v0.2.0
Parts:
- removed J2: Conn_01x04, Connector_PinHeader_2.00mm:PinHeader_1x04_P2.00mm_Vertical, symbol Connector_Generic:Conn_01x04
- added J2: Conn_01x03, Connector_PinHeader_2.54mm:PinHeader_1x03_P2.54mm_Vertical, symbol Connector_Generic:Conn_01x03
Changed lines of the file:
@@
 Title "Zero Cam"
 Date "2021-05-01"
-Rev "v0.1.0"
+Rev "v0.2.0"
 Comp "Juraj Giertl"
 Comment1 "j74a8g@gmail.com"
@@
 $EndComp
 $Comp
-L power:+3.3VA #PWR015
-U 1 1 60893B1B
-P 5250 2650
-F 0 "#PWR015" H 5250 2500 50  0001 C CNN
-F 1 "+3.3VA" H 5265 2823 50  0000 C CNN
-F 2 "" H 5250 2650 50  0001 C CNN
-F 3 "" H 5250 2650 50  0001 C CNN
-	1    5250 2650
-	-1   0    0    -1
-$EndComp
-$Comp
 L Device:C_Small C10
 U 1 1 60896E43
@@
 $EndComp
 Wire Wire Line
-	5250 2650 5250 2750
-Wire Wire Line
-	5150 2850 5150 2750
-Wire Wire Line
-	5150 2750 5250 2750
-Connection ~ 5250 2750
-Wire Wire Line
 	5250 2750 5250 2850
 Wire Wire Line
@@
 	1    0    0    -1
 $EndComp
-$Comp
-L Connector_Generic:Conn_01x04 J2
-U 1 1 60B17D6D
-P 6500 3300
-F 0 "J2" H 6580 3292 50  0000 L CNN
-F 1 "Conn_01x04" H 6580 3201 50  0000 L CNN
-F 2 "Connector_PinHeader_2.00mm:PinHeader_1x04_P2.00mm_Vertical" H 6500 3300 50  0001 C CNN
-F 3 "~" H 6500 3300 50  0001 C CNN
-	1    6500 3300
-	1    0    0    -1
-$EndComp
 Wire Wire Line
 	5850 3300 6300 3300
@@
 $EndComp
 $Comp
-L power:+3.3VA #PWR020
-U 1 1 60B2572E
-P 6300 3200
-F 0 "#PWR020" H 6300 3050 50  0001 C CNN
-F 1 "+3.3VA" V 6315 3327 50  0000 L CNN
-F 2 "" H 6300 3200 50  0001 C CNN
-F 3 "" H 6300 3200 50  0001 C CNN
-	1    6300 3200
-	0    -1   1    0
-$EndComp
-$Comp
 L Device:LED_Small D8
 U 1 1 60B4BF5F
@@
 NoConn ~ 4350 4450
 NoConn ~ 4350 4550
+$Comp
+L Connector_Generic:Conn_01x03 J2
+U 1 1 6096FC1B
+P 6500 3400
+F 0 "J2" H 6580 3442 50  0000 L CNN
+F 1 "Conn_01x03" H 6580 3351 50  0000 L CNN
+F 2 "Connector_PinHeader_2.54mm:PinHeader_1x03_P2.54mm_Vertical" H 6500 3400 50  0001 C CNN
+F 3 "~" H 6500 3400 50  0001 C CNN
+	1    6500 3400
+	1    0    0    -1
+$EndComp
+Wire Wire Line
+	5250 2750 5150 2750
+Wire Wire Line
+	5150 2750 5150 2850
+Connection ~ 5250 2750
+$Comp
+L power:+3.3VA #PWR?
+U 1 1 609A4AF3
+P 5250 2650
+F 0 "#PWR?" H 5250 2500 50  0001 C CNN
+F 1 "+3.3VA" H 5265 2823 50  0000 C CNN
+F 2 "" H 5250 2650 50  0001 C CNN
+F 3 "" H 5250 2650 50  0001 C CNN
+	1    5250 2650
+	1    0    0    -1
+$EndComp
+Wire Wire Line
+	5250 2650 5250 2750
 $EndSCHEMATC
